File: adsb-devboard.kicad_sch (KiCad schematic)
At the start: 89 parts, among them J1 USB_C_Receptacle_USB2.0_16P, J2 Conn_01x20_Pin, J3 Conn_01x20_Pin, J4 Conn_Coaxial, SW1 SW_Push, U1 ICE40UP5K-SG48ITR, U2 RP2350A-QFN60, U3 W25Q128JVP, U4 RT8075ZQW, U5 TJ-S1608SW6TDSLCCYRGB-A5, U6 SPF5189Z, U7 AD8313xRM, U8 TLV3501AID, X1 TA0970B, Y1 Crystal_GND24

Commit message: everything seems ready
Parts:
- C1, C2: value 15p -> 33p
- FB1, FB2, FB3: footprint Inductor_SMD:L_0402_1005Metric -> Inductor_SMD:L_0603_1608Metric
- R23: footprint Resistor_SMD:R_0402_1005Metric -> Resistor_SMD:R_0603_1608Metric
Changed lines of the file:
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@@
 			)
 		)
-		(property "Footprint" "Inductor_SMD:L_0402_1005Metric"
+		(property "Footprint" "Inductor_SMD:L_0603_1608Metric"
 			(at 19.812 196.85 90)
 			(effects
@@
 			)
 		)
-		(property "Footprint" "Resistor_SMD:R_0402_1005Metric"
+		(property "Footprint" "Resistor_SMD:R_0603_1608Metric"
 			(at 64.77 273.558 90)
 			(effects
@@
 			)
 		)
-		(property "Footprint" "Inductor_SMD:L_0402_1005Metric"
+		(property "Footprint" "Inductor_SMD:L_0603_1608Metric"
 			(at 41.402 180.34 90)
 			(effects
@@
 			)
 		)
-		(property "Value" "15p"
+		(property "Value" "33p"
 			(at 257.81 92.7099 0)
 			(effects
@@
 			)
 		)
-		(property "Footprint" "Inductor_SMD:L_0402_1005Metric"
+		(property "Footprint" "Inductor_SMD:L_0603_1608Metric"
 			(at 28.702 160.02 90)
 			(effects
@@
 			)
 		)
-		(property "Value" "15p"
+		(property "Value" "33p"
 			(at 257.81 107.9499 0)
 			(effects

Commit message: sch cleanup and little upgrade
Parts:
- removed L4: 470nH, Inductor_SMD:L_0402_1005Metric, symbol Device:L
- removed TP5, TP6: TestPoint_Alt, TestPoint:TestPoint_Pad_D1.0mm, symbol Connector:TestPoint_Alt
- added C32, C34, C36, C38, C40, C42, C44: 4.7u, Capacitor_SMD:C_0402_1005Metric, symbol Device:C
- added C33, C35, C37, C41, C43, C45, C47, C48: 100n, Capacitor_SMD:C_0402_1005Metric, symbol Device:C
- added C39: 10u, Capacitor_SMD:C_0402_1005Metric, symbol Device:C
- added C46: 1500p, Capacitor_SMD:C_0603_1608Metric, symbol Device:C
- added C49: 2.2u, Capacitor_SMD:C_0603_1608Metric, symbol Device:C
- added C50: 1000p, Capacitor_SMD:C_0603_1608Metric, symbol Device:C
- added C51: 100p, Capacitor_SMD:C_0603_1608Metric, symbol Device:C
- added C52: 1500pf, Capacitor_SMD:C_0603_1608Metric, symbol Device:C
- added C53: 3p, Capacitor_SMD:C_0603_1608Metric, symbol Device:C
- added C54: 200p, Capacitor_SMD:C_0603_1608Metric, symbol Device:C
- added R24, R27, R28: 100, Resistor_SMD:R_0402_1005Metric, symbol Device:R
- added R25, R31: 10K, Resistor_SMD:R_0402_1005Metric, symbol Device:R
- added R26: 2.2K, Resistor_SMD:R_0402_1005Metric, symbol Device:R
- added R29: 53.6, Resistor_SMD:R_0402_1005Metric, symbol Device:R
- added R30: 1K, Resistor_SMD:R_0402_1005Metric, symbol Device:R
- added R32: 100K, Resistor_SMD:R_0402_1005Metric, symbol Device:R
- added U10: SPF5189Z, easyeda2kicad:SOT-343-4_L2.0-W1.3-P1.30-LS2.1-BR, symbol RF_Amplifier:SPF5189Z
- added U11, U9: TCBT-14+, easyeda2kicad:SMD_L3.8-W3.8_TCBT-14, symbol easyeda2kicad:TCBT-14+
- added X2: TA0970B, easyeda2kicad:FILTER-SMD_6P-L3.8-W3.8-P1.27-TL-3, symbol RF_Filter:TA0970B
- C26, C28: value 100p -> 680p
- C29: footprint Capacitor_SMD:C_0402_1005Metric -> Capacitor_SMD:C_0603_1608Metric
- C30: value 1u -> 100n
- C31: value 100p -> 1000p
- R22: value 330 -> 1K
Connections:
- net 1v2: now also C42.1, C43.1, R24.2; no longer U1.29 (VCCPLL)
- net 3v3: now also C29.1, R22.2, C32.1, C33.1, C34.1, C35.1, C36.1, C37.1, C38.1, C39.1, C40.1, C41.1, C49.1, R25.1, R26.1, R27.2, R28.2
- net 3v3_RF: no longer C29.1, FB2.2, FB3.2, U7.1 (VPOS), U7.4 (VPOS)
- net CDONE: now also R26.2
- net CRESETN: now also R25.2
- net GND: now also C32.2, C33.2, C34.2, C35.2, C36.2, C37.2, C38.2, C39.2, C40.2, C41.2, C42.2, C43.2, C44.2, C45.2, C46.2, C47.2, C48.2, C49.2, C52.2, C53.1, C54.1, U10.2 (GND), X2.1 (GND), X2.3 (GND), X2.4 (GND), X2.6 (GND)
- net IO5: now also U8.6; no longer R22.2
- net adout: now also R22.1, R30.2, R31.2; no longer U8.3 (+)
- net smaconn: now also C50.2; no longer C31.2
- net at C30.1, R8.1: now also R32.2; no longer U8.2 (-)
- net at C27.1: now also U9.1 (RF); no longer U6.1
- net at C26.2, U7.2 (INHI): now also R29.1
- net at C28.1, U7.3 (INLO): now also R29.2
- new net: C44.1, C45.1, R24.1, U1.29 (VCCPLL)
- new net: C50.1, U10.3
- new net: C53.2, R30.1, U8.3 (+)
- new net: C54.2, R31.1, R32.1, U8.2 (-)
- new net: C51.1, U11.1 (RF)
- new net 3v3_RF_D: C47.1, C48.1, R27.1, R28.1, U7.1 (VPOS), U7.4 (VPOS)
- new net 3v3_RF_LNA: C46.1, FB3.2, U9.3 (DC)
- new net 3v3_RF_LNA1: C52.1, FB2.2, U11.3 (DC)
- new net biastee: U6.1, U9.2 (RF&DC)
- new net biastee1: U10.1, U11.2 (RF&DC)
- new net firstsawout: C31.2, X2.5 (OUT)
- new net lnaout1: C51.2, X2.2 (IN)
- no-connect marks 2 -> 6
Other:
- note added: "1090Mhz Filters"
- note added: "BANK0"
- note added: "BANK1"
- note added: "BANK2"
- note added: "BIAS TEE"
- note added: "Compartor"
- note added: "Connector"
- note added: "Detector"
- note added: "FLASH"
- note added: "FPGA Power Supply"
- note added: "LNA"
- note added: "PINOUT"
- note added: "Power for RF"
- note added: "RP2350"
- note added: "USB"
- moved on the sheet: C19, C20, C21, C22, C23, C24, C25, C26, C27, C28, C30, C31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

Commit message: upddateeedd schematic
Parts:
- removed R23: 51, Resistor_SMD:R_0603_1608Metric, symbol Device:R
- C27, C51: value 100p -> 12p
Connections:
- net 3v3: now also C49.2; no longer C49.1
- net GND: now also C49.1; no longer C49.2
- net smaconn renamed sma_connector
Other:
- note added: "Filter"
- note added: "RF------>"
- note removed: "1090Mhz Filters"
- moved on the sheet: C26, C27, C28, C29, C30, C31, C47, C48, C49, C50, C51, C52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

Commit message: I HAVE ROUTED THIS FOR THE NTH TIME IDK I HAVE LOST COUNT
Parts:
- removed C27, C51: 12p, Capacitor_SMD:C_0603_1608Metric, symbol Device:C
- removed U11, U9: TCBT-14+, easyeda2kicad:SMD_L3.8-W3.8_TCBT-14, symbol easyeda2kicad:TCBT-14+
- added H1, H3: MountingHole, MountingHole:MountingHole_2.7mm_M2.5, symbol Mechanical:MountingHole
- added L4, L5: HP0603-R10H-N, easyeda2kicad:IND-SMD_L1.6-W1.0, symbol easyeda2kicad:HP0603-R10H-N
- C31: footprint Capacitor_SMD:C_0603_1608Metric -> Capacitor_SMD:C_0402_1005Metric
Connections:
- net lnaout is gone; now on net biastee: X1.2 (IN)
- net lnaout1 is gone; now on net biastee1: X2.2 (IN)
- net 3v3_RF_LNA: now also L5.2
- net 3v3_RF_LNA1: now also L4.2
- net biastee: now also L5.1
- net biastee1: now also L4.1
- no-connect marks 6 -> 2
